Commit message: tracking

File: src/lbr_fri_ros2_stack/lbr_description/urdf/med7/med7_description.xacro (robot description, xacro)
@@ -281,5 +281,6 @@
                 <origin rpy="0 3.14157 0.0" xyz="0.0 0.0 0.0" />
                 <geometry>
-                    <mesh filename="package://lbr_description/meshes/med7/visual/worx+motor+mount+refined+3.stl" scale="0.001 0.001 0.001" />
+                    <!-- <mesh filename="package://lbr_description/meshes/med7/visual/worx+motor+mount+refined+3.stl" scale="0.001 0.001 0.001" /> -->
+                    <mesh filename="package://lbr_description/meshes/med7/visual/ee_mount.stl" scale="0.001 0.001 0.001" />
                 </geometry>
                 <material name="blue">
@@ -290,5 +291,6 @@
                 <origin rpy="0 3.14157 0" xyz="0.0 0.0 0.0" />
                 <geometry>
-                    <mesh filename="package://lbr_description/meshes/med7/collision/worx+motor+mount+refined+3.stl" scale="0.0011 0.0011 0.0011" />
+                    <!-- <mesh filename="package://lbr_description/meshes/med7/collision/worx+motor+mount+refined+3.stl" scale="0.0011 0.0011 0.0011" /> -->
+                    <mesh filename="package://lbr_description/meshes/med7/collision/ee_mount.stl" scale="0.0011 0.0011 0.0011" />
                 </geometry>
             </collision>

Commit message: added a bone scanning trajectory

File: src/lbr_fri_ros2_stack/lbr_description/urdf/med7/med7_description.xacro (robot description, xacro)
@@ -282,5 +282,5 @@
                 <geometry>
                     <!-- <mesh filename="package://lbr_description/meshes/med7/visual/worx+motor+mount+refined+3.stl" scale="0.001 0.001 0.001" /> -->
-                    <mesh filename="package://lbr_description/meshes/med7/visual/ee_mount.stl" scale="0.001 0.001 0.001" />
+                    <mesh filename="package://lbr_description/meshes/med7/visual/mount_with_tip.stl" scale="0.001 0.001 0.001" />
                 </geometry>
                 <material name="blue">
@@ -292,5 +292,5 @@
                 <geometry>
                     <!-- <mesh filename="package://lbr_description/meshes/med7/collision/worx+motor+mount+refined+3.stl" scale="0.0011 0.0011 0.0011" /> -->
-                    <mesh filename="package://lbr_description/meshes/med7/collision/ee_mount.stl" scale="0.0011 0.0011 0.0011" />
+                    <mesh filename="package://lbr_description/meshes/med7/collision/mount_with_tip.stl" scale="0.0011 0.0011 0.0011" />
                 </geometry>
             </collision>
